File: PMS_board/SmoothingConversion.kicad_sch (KiCad schematic)
At the start: 23 parts, among them U15 AP63203WU-7, U7 AP63205QWU7, U9 MIC29300-12WU

Commit message: Add Footprints & such
whoops forgot to push yesterday teehee
Parts:
- C58, C61: footprint (none) -> Capacitor_SMD:C_0603_1608Metric
- U15: footprint SignalStack:AP63203WU-7_DIO -> AP63203WU-7:SO8_DCK_TEX
- U9: footprint TO220-3LD-PL-1_MCH -> MIC29300-12WU:TO220-3LD-PL-1_MCH
Changed lines of the file:
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@@
 			)
 		)
-		(property "Footprint" "TO220-3LD-PL-1_MCH"
+		(property "Footprint" "MIC29300-12WU:TO220-3LD-PL-1_MCH"
 			(at 190.5 44.45 0)
 			(hide yes)
@@
 			)
 		)
-		(property "Footprint" "SignalStack:AP63203WU-7_DIO"
+		(property "Footprint" "AP63203WU-7:SO8_DCK_TEX"
 			(at 189.23 133.35 0)
 			(hide yes)
@@
 			)
 		)
-		(property "Footprint" ""
+		(property "Footprint" "Capacitor_SMD:C_0603_1608Metric"
 			(at 240.9952 53.34 0)
 			(hide yes)
@@
 			)
 		)
-		(property "Footprint" ""
+		(property "Footprint" "Capacitor_SMD:C_0603_1608Metric"
 			(at 187.6552 58.42 0)
 			(hide yes)

Commit message: Minor power changes and new buck for converting to 12V
Changed supply voltage for 3V3 and 5V bucks from 24V to 12V

Changed RoveNode supply from 24V to 12V

Swapped old 12v LDO for buck
Parts:
- removed C58: 10uF, Capacitor_SMD:C_0603_1608Metric, symbol Device:C
- removed C61: 0.1uF, Capacitor_SMD:C_0603_1608Metric, symbol Device:C
- removed U9: MIC29300-12WU, MIC29300-12WU:TO220-3LD-PL-1_MCH, symbol MIC29300-12WU:MIC29300-12WU
- added C2: 22uF, Package_TO_SOT_SMD:TSOT-23-6_HandSoldering, symbol Device:C
- added C3: C, symbol Device:C
- added C4: 22uF, symbol Device:C
- added L3: 18uH, symbol Device:L
- added R10, R4: R_US, symbol Device:R_US
- added U4: DCP3603ACMR, Package_TO_SOT_SMD:TSOT-23-6_HandSoldering, symbol Symbols:DCP3603ACMR
- C47: value 100nF -> 0.1uf
- L2: value 3.9uH -> 3.3uH
- U15: value AP63203WU-7 -> AP63203WU7
Connections:
- net +12V: now also C21.1, D8.2 (A), U7.2 (EN), U7.3 (VIN), C4.1, L3.2, R4.2
- net +24V: no longer C21.1, D8.2 (A), U7.2 (EN), U7.3 (VIN)
- net GND: now also C2.2, C4.2, R10.2, U4.2 (GND)
- new net: C2.1, U4.4 (EN), U4.5 (VIN)
- new net: C3.1, U4.1 (BOOT)
- new net: R10.1, R4.1, U4.3 (FB)
- new net: C3.2, L3.1, U4.6 (SW)
