File: PMS_board/PMS_board.kicad_sch (KiCad schematic)
At the start: 12 parts, among them J17 Conn_01x03_Pin, K1 AZSR190, K2 AZSR190

Commit message: How did our footprints get this geeked???
Parts:
- D14, D15: footprint Package_SON:WSON-8-1EP_6x5mm_P1.27mm_EP3.4x4mm -> (none)
- J17: footprint Converter_DCDC:Converter_DCDC_Cyntec_MUN12AD01-SH -> (none)
- K1, K2: footprint Relay_THT:Relay_SPST-NO_Fujitsu_FTR-LYAA005x_FormA_Vertical -> (none)
Changed lines of the file:
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@@
 			)
 		)
-		(property "Footprint" "Relay_THT:Relay_SPST-NO_Fujitsu_FTR-LYAA005x_FormA_Vertical"
+		(property "Footprint" ""
 			(at 120.65 168.91 0)
 			(hide yes)
@@
 			)
 		)
-		(property "Footprint" "Package_SON:WSON-8-1EP_6x5mm_P1.27mm_EP3.4x4mm"
+		(property "Footprint" ""
 			(at 95.25 167.64 0)
 			(hide yes)
@@
 			)
 		)
-		(property "Footprint" "Relay_THT:Relay_SPST-NO_Fujitsu_FTR-LYAA005x_FormA_Vertical"
+		(property "Footprint" ""
 			(at 163.83 168.91 0)
 			(hide yes)
@@
 			)
 		)
-		(property "Footprint" "Converter_DCDC:Converter_DCDC_Cyntec_MUN12AD01-SH"
+		(property "Footprint" ""
 			(at 21.59 158.75 0)
 			(hide yes)
@@
 			)
 		)
-		(property "Footprint" "Package_SON:WSON-8-1EP_6x5mm_P1.27mm_EP3.4x4mm"
+		(property "Footprint" ""
 			(at 138.43 167.64 0)
 			(hide yes)
