File: PMS_board/VoltageSensing.kicad_sch (KiCad schematic)
At the start: 49 parts, among them J2 BAT_SENSE1, J3 BAT_SENSE2, U1 LM324DR, U19 TS3A27518EIPWRQ1, U2 LM324DR

Commit message: Change based on Will's input
respeced buck
swapped to molex_sls
readded 6-pole switch
Parts:
- removed J2: BAT_SENSE1, Connector_JST:JST_PH_B8B-PH-K_1x08_P2.00mm_Vertical, symbol Connector:Conn_01x08_Pin
- removed J3: BAT_SENSE2, Connector_JST:JST_PH_B8B-PH-K_1x08_P2.00mm_Vertical, symbol Connector:Conn_01x08_Pin
- removed U19: TS3A27518EIPWRQ1, TS3A27518RIPWRQ1:PW24, symbol Symbols:TS3A27518EIPWRQ1
- added J21: BAT_SENSE1, MRDT_Connectors:MOLEX_SL_07_Vertical, symbol Connector:Conn_01x07_Pin
- added J22: BAT_SENSE2, MRDT_Connectors:MOLEX_SL_07_Vertical, symbol Connector:Conn_01x07_Pin
- added U32: EG6201, EG6201:DIP_G6201_EWI, symbol EG6201:EG6201
Connections:
- net GND: now also J21.7 (Pin_7), J22.7 (Pin_7), U32.19, U32.20, U32.21, U32.22
- net COM_CELL1 renamed CELL1
- net CELL1: now also U32.2
- net COM_CELL2 renamed CELL2
- net CELL2: now also U32.5
- net COM_CELL3 renamed CELL3
- net CELL3: now also U32.8
- net COM_CELL4 renamed CELL4
- net CELL4: now also U32.11
- net COM_CELL5 renamed CELL5
- net CELL5: now also U32.14
- net COM_CELL6 renamed CELL6
- net CELL6: now also U32.17
- new net: J21.1 (Pin_1), U32.1
- new net: J21.4 (Pin_4), U32.10
- new net: J22.4 (Pin_4), U32.12
- new net: J21.5 (Pin_5), U32.13
- new net: J22.5 (Pin_5), U32.15
- new net: J21.6 (Pin_6), U32.16
- new net: J22.6 (Pin_6), U32.18
- new net: J22.1 (Pin_1), U32.3
- new net: J21.2 (Pin_2), U32.4
- new net: J22.2 (Pin_2), U32.6
- new net: J21.3 (Pin_3), U32.7
- new net: J22.3 (Pin_3), U32.9
- no-connect marks 3 -> 0
