File: PMS_board/Outputs.kicad_sch (KiCad schematic)
At the start: 87 parts, among them J1 Chopper_Shunt, J20 CORE, J21 DRIVE, J22 JET1, J23 JET2, J24 NET, J25 AUX1, J26 AUX2, J27 D1, J28 D2, J29 D3, J30 D4, J31 T1, J32 T2, J33 T3, J34 T4, Q12 NMOS, Q6 NMOS, U1 VN7140ASTR, U11 VN7007AHTR, U2 VN7140ASTR, U23 VN7007AHTR, U25 TLV7011DCKR, U28 LT1910, U29 IRFS7530TRL7PP, U30 LM74700, U31 LM74700, U8 VN7140ASTR

Commit message: Fixed references
Parts:
- renumbered C54 to C11, C59 to C12, C19 to C13, C24 to C14, C25 to C15, C17 to C16, C18 to C17, C5 to C18, C26 to C19, C28 to C20, C29 to C21, D22 to D13, D20 to D14, D26 to D15, D6 to D16, D7 to D17, D38 to D18, D39 to D19, D40 to D20, D41 to D21, D27 to D22, D42 to D23, J25 to J10, J26 to J11, J27 to J12, J28 to J13, J29 to J14, J30 to J15, J31 to J16, J32 to J17, J33 to J18, J34 to J19, J1 to J4, J20 to J5, J21 to J6, J22 to J7, J23 to J8, J24 to J9, Q6 to Q5, Q12 to Q6, R67 to R50, R68 to R51, R69 to R52, R70 to R53, R20 to R54, R71 to R55, R72 to R56, R75 to R57, R19 to R58, R76 to R59, R77 to R60, R78 to R61, R79 to R62, R73 to R63, R74 to R64, R82 to R65, R83 to R66, R99 to R67, R100 to R68, R101 to R69, R12 to R70, R102 to R71, R106 to R72, R107 to R73, R13 to R74, R14 to R75, R16 to R76, R17 to R77, R18 to R78, R22 to R79, R108 to R80, TP8 to TP14, TP9 to TP15, TP10 to TP16, TP3 to TP17, TP4 to TP18, U1 to U10, U2 to U11, U8 to U12, U23 to U13, U11 to U14, U30 to U15, U25 to U16, U28 to U17, U29 to U18, U31 to U19

Commit message: Divided Bulk Caps
Parts:
- added C37: 1000uF, symbol Device:C_Polarized_US
Connections:
- net GND: now also C37.2
- net Motor_Power2: now also C37.1
Changed lines of the file:
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@@
 	)
 	(junction
+		(at 528.32 81.28)
+		(diameter 0)
+		(color 0 0 0 0)
+	)
+	(junction
 		(at 128.27 82.55)
 		(diameter 0)
@@
 	)
 	(junction
+		(at 521.97 57.15)
+		(diameter 0)
+		(color 0 0 0 0)
+	)
+	(junction
 		(at 336.55 170.18)
 		(diameter 0)
@@
 	(wire
 		(pts
+			(xy 513.08 57.15) (xy 521.97 57.15)
+		)
+		(stroke
+			(width 0)
+			(type default)
+		)
+	)
+	(wire
+		(pts
 			(xy 80.01 119.38) (xy 81.28 119.38)
 		)
@@
 	(wire
 		(pts
+			(xy 521.97 57.15) (xy 521.97 62.23)
+		)
+		(stroke
+			(width 0)
+			(type default)
+		)
+	)
+	(wire
+		(pts
 			(xy 128.27 80.01) (xy 128.27 82.55)
 		)
@@
 	(wire
 		(pts
+			(xy 521.97 81.28) (xy 528.32 81.28)
+		)
+		(stroke
+			(width 0)
+			(type default)
+		)
+	)
+	(wire
+		(pts
 			(xy 541.02 107.95) (xy 541.02 105.41)
 		)
@@
 	(wire
 		(pts
+			(xy 521.97 57.15) (xy 532.13 57.15)
+		)
+		(stroke
+			(width 0)
+			(type default)
+		)
+	)
+	(wire
+		(pts
 			(xy 238.76 91.44) (xy 238.76 96.52)
 		)
@@
 	(wire
 		(pts
-			(xy 532.13 68.58) (xy 532.13 73.66)
+			(xy 532.13 57.15) (xy 532.13 73.66)
 		)
 		(stroke
@@
 	(wire
 		(pts
+			(xy 521.97 69.85) (xy 521.97 81.28)
+		)
+		(stroke
+			(width 0)
+			(type default)
+		)
+	)
+	(wire
+		(pts
 			(xy 485.14 172.72) (xy 485.14 170.18)
 		)
@@
 	)
 	(global_label "Motor_Power2"
+		(shape input)
+		(at 513.08 57.15 180)
+		(fields_autoplaced yes)
+		(effects
+			(font
+				(size 1.27 1.27)
+			)
+			(justify right)
+		)
+		(property "Intersheetrefs" "${INTERSHEET_REFS}"
+			(at 497.0321 57.15 0)
+			(hide yes)
+			(show_name no)
+			(do_not_autoplace no)
+			(effects
+				(font
+					(size 1.27 1.27)
+				)
+				(justify right)
+			)
+		)
+	)
+	(global_label "Motor_Power2"
 		(shape output)
 		(at 336.55 166.37 90)
@@
 	(global_label "Motor_Power2"
 		(shape input)
-		(at 532.13 68.58 90)
-		(fields_autoplaced yes)
-		(effects
-			(font
-				(size 1.27 1.27)
-			)
-			(justify left)
-		)
-		(property "Intersheetrefs" "${INTERSHEET_REFS}"
-			(at 532.13 52.5321 90)
-			(hide yes)
-			(show_name no)
-			(do_not_autoplace no)
-			(effects
-				(font
-					(size 1.27 1.27)
-				)
-				(justify left)
-			)
-		)
-	)
-	(global_label "Motor_Power2"
-		(shape input)
 		(at 238.76 66.04 90)
 		(fields_autoplaced yes)
@@
 					(unit 1)
 				)
+			)
+		)
+	)
+	(symbol
+		(lib_id "Device:C_Polarized_US")
+		(at 521.97 66.04 0)
+		(mirror y)
+		(unit 1)
+		(body_style 1)
+		(exclude_from_sim no)
+		(in_bom yes)
+		(on_board yes)
+		(in_pos_files yes)
+		(dnp no)
+		(property "Reference" "C37"
+			(at 518.16 64.1349 0)
+			(show_name no)
+			(do_not_autoplace no)
+			(effects
+				(font
+					(size 1.27 1.27)
+				)
+				(justify left)
+			)
+		)
+		(property "Value" "1000uF"
+			(at 518.16 66.6749 0)
+			(show_name no)
+			(do_not_autoplace no)
+			(effects
+				(font
+					(size 1.27 1.27)
+				)
+				(justify left)
+			)
+		)
+		(property "Footprint" ""
+			(at 521.97 66.04 0)
+			(hide yes)
+			(show_name no)
+			(do_not_autoplace no)
+			(effects
+				(font
+					(size 1.27 1.27)
+				)
+			)
+		)
+		(property "Datasheet" ""
+			(at 521.97 66.04 0)
+			(hide yes)
+			(show_name no)
+			(do_not_autoplace no)
+			(effects
+				(font
+					(size 1.27 1.27)
+				)
+			)
+		)
+		(property "Description" "Polarized capacitor, US symbol"
+			(at 521.97 66.04 0)
+			(hide yes)
+			(show_name no)
+			(do_not_autoplace no)
+			(effects
+				(font
+					(size 1.27 1.27)
+				)
+			)
+		)
+		(pin "1"
+		)
+		(pin "2"
+		)
+		(instances
+			(project "PMS_board"
+				(path "/282246b0-e0d8-4997-b3ee-58bf10355d52/266cb597-81f7-4ea7-87c1-e1b826fc674e"
+					(reference "C37")
+					(unit 1)
+				)

Commit message: Fixed Bulk caps
Parts:
- added C23, C24, C25, C38: 500uF, symbol Device:C_Polarized_US
Connections:
- net Aux_Power2: now also C23.1
- net Board_Power: now also C25.1
- net GND: now also C23.2, C24.2, C25.2, C38.2
- net Jetson_Power: now also C38.1
- net Network_Power: now also C24.1
