File: PMS_board/PMS_board.kicad_pcb (KiCad board)
At the start: 2 copper layers, 233 parts, among them J1 Conn_01x04_Pin, J10 AUX1, J11 AUX2, J12 D1, J13 D2, J14 D3, J15 D4, J16 T1, J17 T2, J18 T3, J19 T4, J2 BAT_SENSE1, J20 RJ45_LED_Shielded, J23 R_PIs, J3 BAT_SENSE2, J4 Chopper_Shunt, J5 CORE, J6 DRIVE, J7 JET1, J8 JET2, J9 NET, Q7 BSS138, U1 LM324DR, U10 VN7140ASTR, U11 VN7140ASTR, U12 VN7140ASTR, U13 VN7007AHTR, U14 VN7007AHTR, U16 TLV7011DCKR, U17 LT1910, U18 1245HC100-RTR, U19 TS3A27518EIPWRQ1, U2 LM324DR, U20 MCP3204T-CI/ST, U22 AP63203WU7, U23 DCP3603ACMR, U24 AP63205QWU7, U25 IRFS7530TRL7PP, U26 IRFS7530TRL7PP, U27 IRFS7530TRL7PP, U28 LM74800QDRRRQ1, U29 IRFS7530TRL7PP, U30 IRFS7530TRL7PP, U31 LM74800QDRRRQ1, U4 IRFS7530TRL7PP, U5 IRFS7530TRL7PP, U6 LM74800QDRRRQ1, U7 LM74800QDRRRQ1, U8 IRFS7530TRL7PP, U9 IRFS7530TRL7PP

Commit message: Change based on Will's input
respeced buck
swapped to molex_sls
readded 6-pole switch
Parts:
- removed J2: BAT_SENSE1, Connector_JST:JST_PH_B8B-PH-K_1x08_P2.00mm_Vertical
- removed J3: BAT_SENSE2, Connector_JST:JST_PH_B8B-PH-K_1x08_P2.00mm_Vertical
- removed L3: 3.3uH, Inductor_SMD:L_1812_4532Metric_Pad1.30x3.40mm_HandSolder
- removed U19: TS3A27518EIPWRQ1, TS3A27518RIPWRQ1:PW24
- added J21: BAT_SENSE1, MRDT_Connectors:MOLEX_SL_07_Vertical, F.Cu at (-54.1, 53.0)
- added J22: BAT_SENSE2, MRDT_Connectors:MOLEX_SL_07_Vertical, F.Cu at (-54.1, 60.7)
- added L4: 3.9uH, Inductor_SMD:L_1812_4532Metric_Pad1.30x3.40mm_HandSolder, F.Cu at (-211.2, 143.3)
- added U32: EG6201, EG6201:DIP_G6201_EWI, F.Cu at (-64.3, 50.6)
- J1, J7: footprint Connector_JST:JST_PH_B4B-PH-K_1x04_P2.00mm_Vertical -> MRDT_Connectors:MOLEX_SL_04_Vertical
- moved C22 355.3 mm to (-110.6, 55.6)
- moved LCD1 229.7 mm to (-151.6, 182.6)
- moved H3 100.8 mm to (-88.0, 174.3)
- moved H1 100.8 mm to (-102.1, 169.1)
- moved H2 100.8 mm to (-88.0, 166.8)
- moved H4 100.8 mm to (-88.0, 181.9)
- moved J1 12.8 mm to (-59.6, 103.3), turned to 90 degrees
- moved J7 6.63 mm to (205.7, 29.7), turned to 90 degrees
Connections:
- R10 pad 2: COM_CELL4 -> CELL4
- R100 pad 1: COM_CELL6 -> CELL6
- R12 pad 2: COM_CELL3 -> CELL3
- R14 pad 2: COM_CELL2 -> CELL2
- R16 pad 2: COM_CELL1 -> CELL1
- R8 pad 2: COM_CELL5 -> CELL5
