File: PMS_board/PMS_board.kicad_pcb (KiCad board)
At the start: 2 copper layers, 285 parts, among them J1 Conn_01x04_Pin, J10 AUX1, J11 AUX2, J12 D1, J13 D2, J14 D3, J15 D4, J16 T1, J17 T2, J18 T3, J19 T4, J2 BAT_SENSE1, J20 RJ45_LED_Shielded, J3 BAT_SENSE2, J4 Chopper_Shunt, J5 CORE, J6 DRIVE, J7 JET1, J8 JET2, J9 NET, Q1 BSS138, Q2 BSS138, Q3 PMOS, Q4 PMOS, Q7 BSS138, U1 LM324DR, U10 VN7140ASTR, U11 VN7140ASTR, U12 VN7140ASTR, U13 VN7007AHTR, U14 VN7007AHTR, U15 LM324DR, U16 TLV7011DCKR, U17 LT1910, U18 1245HC100-RTR, U19 TS3A27518EIPWRQ1, U2 LM324DR, U20 MCP3204T-CI/ST, U22 AP63203WU7, U23 DCP3603ACMR, U24 AP63205QWU7, U25 IRFS7530TRL7PP, U26 IRFS7530TRL7PP, U27 IRFS7530TRL7PP, U28 LM74800QDRRRQ1, U29 IRFS7530TRL7PP, U3 LM324DR, U30 IRFS7530TRL7PP, U31 LM74800QDRRRQ1, U4 IRFS7530TRL7PP, U5 IRFS7530TRL7PP, U6 LM74800QDRRRQ1, U7 LM74800QDRRRQ1, U8 IRFS7530TRL7PP, U9 IRFS7530TRL7PP

Commit message: Refix Review Work
Parts:
- added J21: Conn_01x02_Pin, Connector_Molex:Molex_Mega-Fit_76829-0002_2x01_P5.70mm_Vertical, F.Cu at (292.7, 135.9)
- added J22: Conn_01x02_Pin, Connector_Molex:Molex_Mega-Fit_76829-0002_2x01_P5.70mm_Vertical, F.Cu at (292.7, 152.0)
- added V4: Jumper_Via, MRDT_Drill_Holes:BATT_PWR_VIA, F.Cu at (311.1, 141.2)
- added V5: Jumper_Via, MRDT_Drill_Holes:BATT_PWR_VIA, F.Cu at (293.6, 175.4)
- H1, H2, H3, H4: footprint MountingHole:MountingHole_3mm_Pad_Via -> MRDT_Drill_Holes:4_40_Hole_Pad_Via
- R83: footprint Footprints:ShuntSMD_BVT-M-R001-1.0 -> Current_Sense:ShuntSMD_BVT-M-R001-1.0
- V1, V2, V3: footprint MRDT_Connectors:MOLEX_UltraFit_02_Vertical -> MRDT_Drill_Holes:BATT_PWR_VIA

Commit message: Uh oh merge conflicts
Parts:
- added J23: R_PIs, Vert_MegaFit:CONN_SD-768290002_02_MOL, F.Cu at (114.0, 87.3)
- J10, J11, J12, J13, J14, J15, J16, J17, J18, J19, J4, J5, J6, J8, J9: footprint MRDT_Connectors:MOLEX_MegaFit_02_Horizontal -> Vert_MegaFit:CONN_SD-768290002_02_MOL
- J7: footprint MRDT_Connectors:MOLEX_MegaFit_02_Horizontal -> Connector_JST:JST_PH_B4B-PH-K_1x04_P2.00mm_Vertical
Connections:
- D3 pad 1: BATT1_SENS6 -> /Microcontroller/VSENSE6
- D4 pad 1: BATT1_SENS5 -> /Microcontroller/VSENSE5
- D5 pad 1: BATT1_SENS4 -> /Microcontroller/VSENSE4
- D6 pad 1: BATT1_SENS3 -> /Microcontroller/VSENSE3
- D7 pad 1: BATT1_SENS2 -> /Microcontroller/VSENSE2
- D8 pad 1: BATT1_SENS1 -> /Microcontroller/VSENSE1
- R10 pad 2: BATT1_CELL4 -> COM_CELL4
- R100 pad 1: BATT1_CELL6 -> COM_CELL6
- R12 pad 2: BATT1_CELL3 -> COM_CELL3
- R14 pad 2: BATT1_CELL2 -> COM_CELL2
- R16 pad 2: BATT1_CELL1 -> COM_CELL1
- R31 pad 2: BATT1_SENS5 -> /Microcontroller/VSENSE5
- R32 pad 2: BATT1_SENS6 -> /Microcontroller/VSENSE6
- R33 pad 2: BATT1_SENS4 -> /Microcontroller/VSENSE4
- R34 pad 2: BATT1_SENS3 -> /Microcontroller/VSENSE3
- R35 pad 2: BATT1_SENS2 -> /Microcontroller/VSENSE2
- R36 pad 2: BATT1_SENS1 -> /Microcontroller/VSENSE1
- R8 pad 2: BATT1_CELL5 -> COM_CELL5
- TP10 pad 1: BATT1_SENS3 -> /Microcontroller/VSENSE3
- TP11 pad 1: BATT1_SENS2 -> /Microcontroller/VSENSE2
- TP12 pad 1: BATT1_SENS1 -> /Microcontroller/VSENSE1
- TP7 pad 1: BATT1_SENS6 -> /Microcontroller/VSENSE6
- TP8 pad 1: BATT1_SENS5 -> /Microcontroller/VSENSE5
- TP9 pad 1: BATT1_SENS4 -> /Microcontroller/VSENSE4
- U19 pad 1: BATT1_SENS2 -> BATT1_CELL2
- U19 pad 10: /Microcontroller/VSENSE5 -> COM_CELL5
- U19 pad 11: BATT2_SENS1 -> BATT2_CELL1
- U19 pad 12: /Microcontroller/VSENSE6 -> COM_CELL6
- U19 pad 13: BATT2_SENS2 -> BATT2_CELL2
- U19 pad 14: /Voltage Sensing/SW2 -> /Voltage Sensing/CELL_SW
- U19 pad 15: BATT2_SENS3 -> BATT2_CELL3
- U19 pad 16: BATT2_SENS6 -> BATT2_CELL6
- U19 pad 17: BATT2_SENS4 -> BATT2_CELL4
- U19 pad 18: BATT2_SENS5 -> BATT2_CELL5
- U19 pad 19: BATT1_SENS5 -> BATT1_CELL5
- U19 pad 2: BATT1_SENS1 -> BATT1_CELL1
- U19 pad 21: BATT1_SENS4 -> BATT1_CELL4
- U19 pad 22: BATT1_SENS6 -> BATT1_CELL6
- U19 pad 23: BATT1_SENS3 -> BATT1_CELL3
- U19 pad 24: /Voltage Sensing/SW1 -> /Voltage Sensing/CELL_SW
- U19 pad 4: /Microcontroller/VSENSE1 -> COM_CELL1
- U19 pad 6: /Microcontroller/VSENSE2 -> COM_CELL2
- U19 pad 7: /Microcontroller/VSENSE3 -> COM_CELL3
- U19 pad 9: /Microcontroller/VSENSE4 -> COM_CELL4

Commit message: Layouted Voltage sensing + OR'ing circuit
Parts:
- D10, D11, D28, D29: value PTVS26VZ1USK -> BZX84C15LT1G; footprint Diode_SMD:Nexperia_DSN1608-2_1.6x0.8mm -> BZX84C15LT1G:SOT95P240X111-3N
- moved Q1 602.8 mm to (-136.7, -236.2)
- moved Q2 602.8 mm to (-136.7, -231.7)
- moved Q3 602.8 mm to (-153.4, -250.1)
- moved Q4 602.8 mm to (-153.4, -242.3)
- moved R1 602.8 mm to (-131.7, -252.8)
- moved R2 602.8 mm to (-131.7, -250.2)
- moved D1 597.3 mm to (-156.4, -210.5)
- moved D2 597.3 mm to (-151.5, -210.5)
- moved R3 597.3 mm to (-142.2, -220.6)
- moved R4 597.3 mm to (-142.2, -218.0)
- moved R5 597.3 mm to (-142.2, -215.5)
- moved R6 597.3 mm to (-142.2, -213.0)
- moved J22 526.5 mm to (-151.7, -130.3)
- moved J21 502.6 mm to (-133.5, -130.5)
- moved J2 405.5 mm to (124.5, -138.4)
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
Commit message: Aux Ideal diode *very* rough layout
Parts:
- moved D12 349.4 mm to (47.0, 276.8)
- moved D13 349.4 mm to (51.9, 276.8)
- moved D14 349.4 mm to (56.8, 276.8)
- moved D16 349.4 mm to (54.7, 257.4)
- moved D18 349.4 mm to (54.7, 262.6)
- moved D21 349.4 mm to (54.7, 270.4)
- moved TP17 349.4 mm to (58.4, 266.8)
- moved TP18 349.4 mm to (58.4, 269.8)
- moved U11 349.4 mm to (48.2, 266.1)
- moved U12 349.4 mm to (48.2, 272.8)
- moved U13 349.4 mm to (48.0, 248.7)
- moved U14 349.4 mm to (56.3, 248.7)
- moved C16 349.4 mm to (45.9, 282.4)
- moved D17 349.4 mm to (54.7, 260.0)
- moved D19 349.4 mm to (54.7, 265.2)
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Other:
- board text added: "Aux Ideal Diode"
- board text added: "OR'ing"
- board text added: "VSENSE"

Commit message: I am in layout hell.
Parts:
- removed D1, D2: D_Zener, MRDT_Passives:SOT-23_Diode
- removed D15, D22, D30, D31, D32, D33: BZV55B3V3, Diode_SMD:D_MiniMELF
- removed J21, J22: Conn_01x02_Pin, Connector_Molex:Molex_Mega-Fit_76829-0002_2x01_P5.70mm_Vertical
- removed Q1, Q2: BSS138, Package_TO_SOT_SMD:SOT-23
- removed Q3, Q4: PMOS, Package:SQL147
- removed R101, R102, R11, R13, R15, R17, R9: 54.9k, Resistor_SMD:R_0603_1608Metric_Pad0.98x0.95mm_HandSolder
- removed R103, R104, R105, R106, R107, R108, R109, R110, R111, R112, R113, R114: 39.2k, Resistor_SMD:R_0603_1608Metric_Pad0.98x0.95mm_HandSolder
- removed R115, R116, R117, R118, R119, R120: 1k, Resistor_SMD:R_0603_1608Metric_Pad0.98x0.95mm_HandSolder
- removed R4, R6: 22k, Resistor_SMD:R_0603_1608Metric_Pad0.98x0.95mm_HandSolder
- removed R5: 10k, Resistor_SMD:R_0603_1608Metric_Pad0.98x0.95mm_HandSolder
- removed TP19, TP2, TP20, TP21, TP22, TP23, TP24, TP25, TP26, TP27, TP3, TP6: TestPoint, TestPoint:TestPoint_Pad_D1.0mm
- removed U15, U3: LM324DR, Package_SO:SOIC-14_3.9x8.7mm_P1.27mm
- removed V4: Jumper_Via, MRDT_Drill_Holes:BATT_PWR_VIA
- D10, D11, D28, D29: value BZX84C15LT1G -> MMSZ5264BT1G; footprint BZX84C15LT1G:SOT95P240X111-3N -> Diode_SMD:D_SOD-123
- J1: footprint MRDT_Connectors:MOLEX_SL_04_Horizontal -> Connector_JST:JST_PH_B4B-PH-K_1x04_P2.00mm_Vertical
- R1, R2: value 100k -> 10k
- R3: value 10k -> 1m; footprint Resistor_SMD:R_0603_1608Metric_Pad0.98x0.95mm_HandSolder -> Current_Sense:ShuntSMD_BVT-M-R001-1.0
- U17: footprint Package_DFN_QFN:DFN-24-1EP_4x7mm_P0.5mm_EP2.64x6.44mm -> Package_SO:SO-8_3.9x4.9mm_P1.27mm
- moved D27 606.8 mm to (-206.2, 138.7)
- moved C26 606.4 mm to (-225.2, 135.9)
- moved C31 606.4 mm to (-220.9, 135.9)
- moved C34 606.4 mm to (-220.9, 143.4)
- moved C36 606.4 mm to (-216.5, 135.9)
- moved D26 606.4 mm to (-203.0, 142.9)
- moved L3 606.4 mm to (-210.7, 143.3)
- moved R88 606.4 mm to (-216.5, 138.4)
- moved D25 602.4 mm to (-220.8, 146.8)
- moved U22 597.4 mm to (-211.4, 138.1)
- moved U23 578.7 mm to (-176.5, 139.2)
- moved C27 573.1 mm to (-191.7, 139.3)
- moved C29 573.1 mm to (-191.7, 144.3)
- moved C32 573.1 mm to (-187.3, 139.3)
- moved R89 573.1 mm to (-183.0, 141.8)
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Connections:
- J1 pad 3: Net-(J1-Pin_3) -> ESTOP1
- J1 pad 4: Net-(J1-Pin_4) -> ESTOP2
- J7 pad 2: +3V3 -> +3V3 (Jetson)
- R1 pad 1: BATTERY_IN2 -> ESTOP1
- R1 pad 2: Net-(Q1-D) -> GND
- R2 pad 1: BATTERY_IN1 -> ESTOP2
- R2 pad 2: Net-(Q2-D) -> GND
- R3 pad 1: Net-(J1-Pin_4) -> /HotSwap/Aalmout
- R3 pad 2: ESTOP1 -> /Current Sensing/BATT_OUT
- R43 pad 2: VBATT2 -> BATTERY_IN2
- R48 pad 2: VBATT1 -> BATTERY_IN1
- R84 pad 1: Net-(R83-Pad2) -> /HotSwap/Aalmout
- R85 pad 1: Net-(R83-Pad3) -> /Current Sensing/BATT_OUT
- U4 pad 8: VBATT2 -> BATTERY_IN2
- U6 pad 6: /HotSwap/vsnsB -> ESTOP2
- U7 pad 6: /HotSwap/vsnsA -> ESTOP1
- U9 pad 8: VBATT1 -> BATTERY_IN1
Routing:
- added copper zone on B.Cu, net Aux_Power2
- added copper zone on F.Cu, net Aux_Power2
- added copper zone on B.Cu, net Board_Power
- added copper zone on F.Cu, net Board_Power
- added copper zone on B.Cu, net Jetson_Power
- added copper zone on F.Cu, net Jetson_Power
- added copper zone on B.Cu, net Motor_Power2
- added copper zone on F.Cu, net Motor_Power2
- added copper zone on B.Cu, net Network_Power
- added copper zone on F.Cu, net Network_Power
Other:
- board text added: "12V Converter"
- board text added: "3V3 Converter"
- board text added: "5V Converter"
- board text added: "Buzzer"
- board text added: "Load Switching"
- board text removed: "Aux Ideal Diode"

Commit message: Really rough layout
Parts:
- moved H4 412.1 mm to (271.1, 25.2)
- moved J20 361.2 mm to (248.3, 19.7)
- moved H3 342.7 mm to (270.8, 163.1)
- moved D3 329.0 mm to (248.4, 70.5)
- moved D4 329.0 mm to (251.4, 82.7)
- moved D5 329.0 mm to (250.9, 112.0)
- moved D6 329.0 mm to (232.1, 86.8)
- moved D7 329.0 mm to (240.8, 66.5)
- moved J2 329.0 mm to (268.7, 74.9)
- moved J3 329.0 mm to (268.8, 96.1)
- moved R10 329.0 mm to (247.9, 85.9)
- moved R14 329.0 mm to (243.8, 102.4)
- moved R18 329.0 mm to (235.2, 77.1)
- moved R19 329.0 mm to (243.8, 69.5)
- moved R20 329.0 mm to (244.8, 72.6)
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Routing:
- added copper zone on B.Cu, net BATTERY_IN1
- added copper zone on F.Cu, net BATTERY_IN1
- added copper zone on B.Cu, net BATTERY_IN2
- added copper zone on F.Cu, net BATTERY_IN2
Other:
- board outline added: 249.9 x 145.8 mm
- board text removed: "Load Switching"
