File: PMS_board/PMS_board.kicad_pcb (KiCad board)
At the start: 2 copper layers, 249.9 x 145.8 mm, 239 parts, among them J1 Conn_01x04_Pin, J10 AUX1, J11 AUX2, J12 D1, J13 D2, J14 D3, J15 D4, J16 T1, J17 T2, J18 T3, J19 T4, J2 BAT_SENSE1, J20 RJ45_LED_Shielded, J21 BAT_SENSE1, J22 BAT_SENSE2, J23 R_PIs, J3 BAT_SENSE2, J4 Chopper_Shunt, J5 CORE, J6 DRIVE, J7 JET1, J8 JET2, J9 NET, Q7 BSS138, U1 LM324DR, U10 VN7140ASTR, U11 VN7140ASTR, U12 VN7140ASTR, U13 VN7007AHTR, U14 VN7007AHTR, U16 TLV7011DCKR, U17 LT1910, U18 1245HC100-RTR, U19 TS3A27518EIPWRQ1, U2 LM324DR, U20 MCP3204T-CI/ST, U22 AP63203WU7, U23 DCP3603ACMR, U24 AP63205QWU7, U25 IRFS7530TRL7PP, U26 IRFS7530TRL7PP, U27 IRFS7530TRL7PP, U28 LM74800QDRRRQ1, U29 IRFS7530TRL7PP, U30 IRFS7530TRL7PP, U31 LM74800QDRRRQ1, U32 EG6201, U4 IRFS7530TRL7PP, U5 IRFS7530TRL7PP, U6 LM74800QDRRRQ1, U7 LM74800QDRRRQ1, U8 IRFS7530TRL7PP, U9 IRFS7530TRL7PP

Commit message: Fixed layout after some merge hoopla
Parts:
- removed the J1 at (-58.9, 90.5)
- removed the J1 at (-59.6, 103.3)
- removed J2: BAT_SENSE1, Connector_JST:JST_PH_B8B-PH-K_1x08_P2.00mm_Vertical
- removed J3: BAT_SENSE2, Connector_JST:JST_PH_B8B-PH-K_1x08_P2.00mm_Vertical
- removed the J7 at (206.3, 23.1)
- removed the J7 at (205.7, 29.7)
- removed U19: TS3A27518EIPWRQ1, TS3A27518RIPWRQ1:PW24
- added J1: Conn_01x04_Pin, MRDT_Connectors:MOLEX_SL_04_Vertical, F.Cu at (142.7, 162.1)
- added J7: JET1, MRDT_Connectors:MOLEX_SL_04_Vertical, F.Cu at (203.3, 33.5)
- moved H3 407.1 mm to (270.8, 25.4)
- moved H2 340.0 mm to (270.3, 163.1)
- moved J21 330.1 mm to (269.7, 117.3), turned to 90 degrees
- moved U32 326.6 mm to (260.5, 85.5)
- moved J22 325.0 mm to (270.3, 81.8), turned to 90 degrees
- moved C22 320.7 mm to (247.5, 51.3)
- moved LCD1 319.7 mm to (219.5, 103.1), turned to -90 degrees
- moved L4 285.4 mm to (74.0, 131.6)
- moved L3 273.7 mm to (63.0, 141.2)
- moved H4 265.5 mm to (28.8, 25.2)
- moved H1 140.9 mm to (29.0, 163.1)
- moved R41 7.18 mm to (226.5, 103.0)
- moved D5 7.18 mm to (243.8, 112.6)
- moved D9 7.18 mm to (227.0, 99.4)
- moved R12 7.18 mm to (240.2, 111.6)
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Other:
- board text removed: "OR'ing"

Commit message: Moved some things around
Parts:
- moved C28 152.0 mm to (190.1, 76.1), turned to 180 degrees
- moved C30 148.9 mm to (190.1, 71.1), turned to 180 degrees
- moved C33 146.6 mm to (185.8, 76.1), turned to 180 degrees
- moved C35 143.4 mm to (185.8, 71.1), turned to 180 degrees
- moved U24 137.0 mm to (179.2, 74.0), turned to 180 degrees
- moved L2 122.9 mm to (167.5, 74.0), turned to 180 degrees
- moved C26 122.6 mm to (164.9, 88.7)
- moved C31 122.6 mm to (169.2, 88.7)
- moved C36 122.6 mm to (173.6, 88.7)
- moved D25 122.6 mm to (169.3, 99.6)
- moved D26 122.6 mm to (187.1, 95.7)
- moved R88 122.6 mm to (173.6, 91.2)
- moved U22 122.6 mm to (178.7, 90.8)
- moved C34 122.6 mm to (169.2, 96.2)
- moved L3 122.6 mm to (177.3, 96.9)
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Other:
- board text removed: "12V Converter"
- board text removed: "3V3 Converter"
- board text removed: "5V Converter"

Commit message: Routed ORing circuit. (Please don't make me redo this)
Parts:
- removed R83: 1m, Current_Sense:ShuntSMD_BVT-M-R001-1.0
- moved U18 138.3 mm to (-56.0, 96.3)
- moved C12 138.3 mm to (-42.3, 94.2)
- moved C1 86.0 mm to (119.9, 128.3), turned to -90 degrees
- moved C5 85.3 mm to (119.1, 119.1), turned to 180 degrees
- moved C3 78.1 mm to (113.3, 120.7)
- moved R42 73.0 mm to (122.9, 127.8), turned to 180 degrees
- moved C4 67.1 mm to (100.8, 128.5), turned to 90 degrees
- moved U5 63.1 mm to (132.3, 111.5), turned to 0 degrees
- moved C2 58.8 mm to (125.2, 123.2), turned to -90 degrees
- moved C9 46.9 mm to (78.7, 123.7), turned to -90 degrees
- moved R3 45.9 mm to (116.6, 103.1), turned to 90 degrees
- moved C6 42.4 mm to (76.7, 116.8), turned to 180 degrees
- moved R49 38.9 mm to (77.2, 128.8), turned to 180 degrees
- moved C10 38.6 mm to (73.2, 128.3), turned to 180 degrees
- moved U7 35.4 mm to (72.4, 124.2)
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Routing:
- net ESTOP2: track 0.00 -> 65.0 mm, vias 0 -> 1
- net ESTOP1: track 0.00 -> 63.6 mm, vias 0 -> 1
- net /HotSwap/Aalmout: track 0.00 -> 42.3 mm
- net /HotSwap/vsnsB: track 0.00 -> 37.2 mm, vias 0 -> 3
- net /HotSwap/vsnsA: track 0.00 -> 33.8 mm, vias 0 -> 3
- net /HotSwap/sourceA: track 0.00 -> 25.7 mm, vias 0 -> 2
- net /HotSwap/HGateB: track 0.00 -> 22.7 mm
- net /HotSwap/HGateA: track 0.00 -> 19.8 mm
- net /HotSwap/sourceB: track 0.00 -> 14.0 mm, vias 0 -> 2
- net /HotSwap/DGateB: track 0.00 -> 12.0 mm, vias 0 -> 2
- net /HotSwap/DGateA: track 0.00 -> 11.7 mm, vias 0 -> 2
- net Net-(U6-OV): track 0.00 -> 8.19 mm
- net Net-(U7-OV): track 0.00 -> 8.11 mm
- net Net-(U6-CAP): track 0.00 -> 5.30 mm
- net Net-(U7-CAP): track 0.00 -> 5.22 mm
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- added copper zone on F.Cu, net /HotSwap/Aalmout
- added copper zone on F.Cu, net /HotSwap/sourceA
- added copper zone on F.Cu, net /HotSwap/sourceB

Commit message: Routed AUX rail and Vsense
Parts:
- moved U18 174.6 mm to (118.6, 98.8), turned to 180 degrees
- moved C12 150.5 mm to (107.7, 81.8), turned to 0 degrees
- moved C32 93.1 mm to (264.9, 120.9)
- moved L1 93.1 mm to (242.3, 118.9)
- moved U23 93.1 mm to (254.0, 120.9)
- moved C27 93.1 mm to (269.2, 120.9)
- moved C29 93.1 mm to (269.2, 115.9)
- moved R89 93.1 mm to (260.5, 118.4)
- moved R90 93.1 mm to (260.5, 115.9)
- moved R85 78.1 mm to (136.9, 103.4)
- moved C26 77.0 mm to (241.8, 91.9)
- moved C31 77.0 mm to (246.2, 91.9)
- moved C34 77.0 mm to (246.2, 99.4)
- moved D27 77.0 mm to (260.9, 94.6)
- moved L3 77.0 mm to (254.3, 100.1)
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Routing:
- net Net-(U1C-+): track 0.00 -> 113.6 mm, vias 0 -> 2
- net Net-(U1C--): track 0.00 -> 84.2 mm
- net +24V: track 0.00 -> 77.5 mm, vias 0 -> 3
- net Net-(U1B-+): track 0.00 -> 74.6 mm
- net GND: track 0.00 -> 71.9 mm, vias 0 -> 39
- net /Current Sensing/Aux_Sense: track 0.00 -> 68.3 mm, vias 0 -> 2
- net /Current Sensing/Total_Curr: track 0.00 -> 63.7 mm
- net Net-(U1D--): track 0.00 -> 60.3 mm, vias 0 -> 2
- net /Microcontroller/VSENSE4: track 0.00 -> 56.9 mm, vias 0 -> 1
- net /Microcontroller/VSenseT: track 0.00 -> 50.5 mm
- net /Microcontroller/VSENSE5: track 0.00 -> 49.4 mm, vias 0 -> 2
- net /Microcontroller/VSENSE6: track 0.00 -> 47.7 mm, vias 0 -> 2
- net Net-(J21-Pin_2): track 0.00 -> 46.1 mm
- net Net-(J22-Pin_4): track 0.00 -> 43.5 mm
- net Net-(J21-Pin_1): track 0.00 -> 42.9 mm
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- added copper zone on F.Cu, net +24V
- added copper zone on F.Cu, net /Load Switching + Outputs/sourceC
- added copper zone on F.Cu, net Aux_Power1
- added copper zone on B.Cu, net GND
Other:
- board text removed: "Buzzer"
- board text removed: "VSENSE"
